Commit message: Move ee_link to center of attached calibration object

File: ur_description/urdf/ur5.urdf.xacro (robot description, xacro)
@@ -276,5 +276,5 @@
       <parent link="${prefix}wrist_3_link" />
       <child link = "${prefix}ee_link" />
-      <origin xyz="0.0 ${wrist_3_length} 0.0" rpy="0.0 0.0 ${pi/2.0}" />
+      <origin xyz="-0.12 ${wrist_3_length} 0.12" rpy="${pi/4.0} 0.0 ${pi/2.0}" />
     </joint>
     <link name="${prefix}ee_link">
